File: kicad/data_logger_load_cell/data_logger_load_cell.kicad_sch (KiCad schematic)
At the start: 12 parts, among them SW1 SW_SPDT_312

Commit message: Updates to schematics
Connections:
- net +3V3: now also U1. (33)
- net at U5. (VIN-): now also SW1.2 (C); no longer U1. (33)
- new net: U1. (33), U5. (VIN-)
- new net: U2. (VCC), U6. (SIGNAL_W) (x2)
- new net: U11. (SIGNAL_W), U12. (VCC) (x2)
- new net: U10. (VCC), U9. (SIGNAL_W) (x2)
Changed lines of the file:
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@@
+	(symbol
+		(lib_id "power:+3V3")
+		(at 166.37 73.66 270)
+		(unit 1)
+		(exclude_from_sim no)
+		(in_bom yes)
+		(on_board yes)
+		(dnp no)
+		(fields_autoplaced yes)
+		(property "Reference" "#PWR02"
+			(at 162.56 73.66 0)
+			(effects
+				(font
+					(size 1.27 1.27)
+				)
+				(hide yes)
+			)
+		)
+		(property "Value" "+3V3"
+			(at 170.18 73.6599 90)
+			(effects
+				(font
+					(size 1.27 1.27)
+				)
+				(justify left)
+			)
+		)
+		(property "Footprint" ""
+			(at 166.37 73.66 0)
+			(effects
+				(font
+					(size 1.27 1.27)
+				)
+				(hide yes)
+			)
+		)
+		(property "Datasheet" ""
+			(at 166.37 73.66 0)
+			(effects
+				(font
+					(size 1.27 1.27)
+				)
+				(hide yes)
+			)
+		)
+		(property "Description" "Power symbol creates a global label with name \"+3V3\""
+			(at 166.37 73.66 0)
+			(effects
+				(font
+					(size 1.27 1.27)
+				)
+				(hide yes)
+			)
+		)
+		(pin "1"
+		)
+		(instances
+			(project ""
+				(path "/b0934bd5-4378-4212-89da-83cc5020f03e"
+					(reference "#PWR02")
+					(unit 1)
+				)
+			)
+		)
+	)
 	(symbol
 		(lib_id "power:+3V3")

Commit message: Updating the schematics to correctly show the connections
Connections:
- net pin_13: no longer U12. (VCC)
- net pin_2: now also U10. (VCC); no longer U2. (VCC)
- net pin_3: now also U12. (VCC); no longer U10. (VCC)
- net pin_4: now also U2. (VCC); no longer U12. (VCC)
- net at U5. (VIN-): now also SW1.2 (C); no longer U1. (33)
- net pin_33: now reaches U12. (VCC)
- new net: U1. (33), U5. (VIN-)
- new net: U2. (VCC), U6. (SIGNAL_W) (x2)
- new net: U11. (SIGNAL_W), U12. (VCC) (x2)
- new net: U10. (VCC), U9. (SIGNAL_W) (x2)
Changed lines of the file:
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@@
+	(wire
+		(pts
+			(xy 147.32 78.74) (xy 148.59 78.74)
+		)
+		(stroke
+			(width 0)
+			(type default)
+		)
+	)
+	(wire
+		(pts
+			(xy 59.69 133.35) (xy 87.63 133.35)
+		)
+		(stroke
+			(width 0)
+			(type default)
+		)
+	)
+	(wire
+		(pts
+			(xy 217.17 71.12) (xy 217.17 83.82)
+		)
+		(stroke
+			(width 0)
+			(type default)
+		)
+	)
+	(wire
+		(pts
+			(xy 240.03 81.28) (xy 240.03 88.9)
+		)
+		(stroke
+			(width 0)
+			(type default)
+		)
+	)
 	(wire
 		(pts
@@
 	(wire
 		(pts
-			(xy 147.32 78.74) (xy 148.59 78.74)
-		)
-		(stroke
-			(width 0)
-			(type default)
-		)
-	)
-	(wire
-		(pts
-			(xy 59.69 133.35) (xy 87.63 133.35)
-		)
-		(stroke
-			(width 0)
-			(type default)
-		)
-	)
-	(wire
-		(pts
-			(xy 217.17 71.12) (xy 217.17 83.82)
-		)
-		(stroke
-			(width 0)
-			(type default)
-		)
-	)
-	(wire
-		(pts
-			(xy 240.03 81.28) (xy 240.03 88.9)
-		)
-		(stroke
-			(width 0)
-			(type default)
-		)
-	)
-	(wire
-		(pts
 			(xy 124.46 63.5) (xy 115.57 63.5)
 		)
@@
 		)
 	)
-	(label "pin_13"
+	(label "pin_3"
 		(at 124.46 133.35 0)
 		(effects
@@
 		)
 	)
-	(label "pin_3"
+	(label "pin_14"
 		(at 123.19 95.25 0)
 		(effects
@@
 		)
 	)
-	(label "pin_4"
+	(label "pin_33"
 		(at 124.46 130.81 0)
 		(effects
@@
 		)
 	)
+	(label "pin_4"
+		(at 124.46 66.04 0)
+		(effects
+			(font
+				(size 1.27 1.27)
+			)
+			(justify left bottom)
+		)
+	)
 	(label "pin_15"
-		(at 124.46 66.04 0)
-		(effects
-			(font
-				(size 1.27 1.27)
-			)
-			(justify left bottom)
-		)
-	)
-	(label "pin_2"
 		(at 124.46 63.5 0)
 		(effects
@@
 		)
 	)
-	(label "pin_4"
-		(at 124.46 130.81 0)
-		(effects
-			(font
-				(size 1.27 1.27)
-			)
-			(justify left bottom)
-		)
-	)
-	(label "pin_14"
+	(label "pin_2"
 		(at 123.19 97.79 0)
 		(effects
